Commit message: launched rviz

File: diff_drive/urdf/ddrive.gazebo.xacro (robot description, xacro)
@@ -41,4 +41,5 @@
         <minDepth>0.001</minDepth>
         <maxVel>1.0</maxVel>
+        <material>Gazebo/FlatBlack</material>
     </gazebo>
   <!-- <gazebo reference="caster_top_back_link">
@@ -59,7 +60,8 @@
         <minDepth>0.001</minDepth>
         <maxVel>1.0</maxVel>
+        <material>Gazebo/FlatBlack</material>
     </gazebo>
-  <gazebo>
-    <plugin name="ddrive_controller" filename="libgazebo_ros_diff_drive.so">
+  <!-- <gazebo>
+    <plugin name="differential_drive_controller" filename="libgazebo_ros_diff_drive.so">
       <commandTopic>cmd_vel</commandTopic>
       <odometryTopic>odom</odometryTopic>
@@ -83,4 +85,27 @@
       <rosDebugLevel>na</rosDebugLevel>
     </plugin>
+  </gazebo> -->
+  <gazebo>
+    <plugin name="differential_drive_controller" filename="libgazebo_ros_diff_drive.so">
+      <rosDebugLevel>na</rosDebugLevel>
+      <alwaysOn>true</alwaysOn>
+      <updateRate>100</updateRate>
+      <leftJoint>wheel_left_joint</leftJoint>
+      <rightJoint>wheel_right_joint</rightJoint>
+      <wheelSeparation>0.5045</wheelSeparation>
+      <wheelDiameter>0.017</wheelDiameter>
+      <wheelTorque>10</wheelTorque>
+      <commandTopic>diff/cmd_vel</commandTopic>
+      <odometryTopic>diff/odom</odometryTopic>
+      <odometryFrame>odom</odometryFrame>
+      <!-- <robotBaseFrame>base_link</robotBaseFrame> -->
+      <publishWheelTF>false</publishWheelTF>
+      <publishOdomTF>true</publishOdomTF>
+      <robotBaseFrame>base_footprint</robotBaseFrame>
+      <publishWheelJointState>true</publishWheelJointState>
+      <wheelAcceleration>false</wheelAcceleration>
+      <odometrySource>world</odometrySource>
+      <publishTf>true</publishTf>
+    </plugin>
   </gazebo>
 </robot>

File: diff_drive/urdf/ddrive.urdf.xacro (robot description, xacro)
@@ -1,7 +1,6 @@
 <?xml version="1.0"?>
 <robot name="ddrive" xmlns:xacro="http://www.ros.org/wiki/xacro">
-  <!-- <xacro:include filename="$(find turtlebot3_description)/urdf/common_properties.xacro"/>
-  <xacro:include filename="$(find turtlebot3_description)/urdf/turtlebot3_burger.gazebo.xacro"/> -->
-  <xacro:property name="ddrive" value="$(find diff_drive)/config/ddrive.yaml" />
+  <xacro:include filename="$(find diff_drive)/urdf/ddrive.gazebo.xacro"/>
+  <xacro:property name="ddrive" value="$(find diff_drive)/config/ddrive.yaml"/>
   <xacro:property name="dictionary" value="${load_yaml(ddrive)}"/>
   <xacro:property name="L" value="${dictionary['L']}"/>
@@ -95,9 +94,9 @@
     <parent link="base_link"/>
     <child link="caster_bottom_back_link"/>
-    <origin xyz="${-3*L/7} 0 ${-H/2 - 0.030}" rpy="-1.57 0 0"/>
+    <origin xyz="${-3*L/7} 0 ${-H/2 - 0.026}" rpy="-1.57 0 0"/>
   </joint>
   <link name="caster_bottom_back_link">
     <visual>
-      <origin rpy="1.57 0 0" xyz="0 0.001 0"/>
+      <origin rpy="1.57 0 0" xyz="0 0 0"/>
       <geometry>
         <sphere radius="0.03"/>
@@ -106,5 +105,5 @@
     </visual>
     <collision>
-      <origin rpy="1.57 0 0" xyz="0 0.001 0"/>
+      <origin rpy="1.57 0 0" xyz="0 0 0"/>
       <geometry>
         <sphere radius="0.03"/>
@@ -122,9 +121,9 @@
     <parent link="base_link"/>
     <child link="caster_top_back_link"/>
-    <origin xyz="${-3*L/7} 0 ${H/2 + 0.030}" rpy="-1.57 0 0"/>
+    <origin xyz="${-3*L/7} 0 ${H/2 + 0.026}" rpy="-1.57 0 0"/>
   </joint>
   <link name="caster_top_back_link">
     <visual>
-      <origin rpy="1.57 0 0" xyz="0 0.001 0"/>
+      <origin rpy="1.57 0 0" xyz="0 0 0"/>
       <geometry>
         <sphere radius="0.03"/>
@@ -133,5 +132,5 @@
     </visual>
     <collision>
-      <origin rpy="1.57 0 0" xyz="0 0.001 0"/>
+      <origin rpy="1.57 0 0" xyz="0 0 0"/>
       <geometry>
         <sphere radius="0.03"/>

Commit message: fixed bugs on model. node makes the robot to move

File: diff_drive/urdf/ddrive.gazebo.xacro (robot description, xacro)
@@ -5,6 +5,6 @@
   </gazebo>
   <gazebo reference="wheel_left_link">
-    <mu1>0.1</mu1>
-    <mu2>0.1</mu2>
+    <mu1>0.3</mu1>
+    <mu2>0.3</mu2>
     <kp>500000.0</kp>
     <kd>10.0</kd>
@@ -15,6 +15,6 @@
   </gazebo>
   <gazebo reference="wheel_right_link">
-    <mu1>0.1</mu1>
-    <mu2>0.1</mu2>
+    <mu1>0.3</mu1>
+    <mu2>0.3</mu2>
     <kp>500000.0</kp>
     <kd>10.0</kd>
@@ -24,66 +24,22 @@
     <material>Gazebo/FlatBlack</material>
   </gazebo>
-  <!-- <gazebo reference="caster_bottom_back_link">
-    <mu1>0.1</mu1>
-    <mu2>0.1</mu2>
+  <gazebo reference="caster_bottom_back_link">
+    <mu1>0.0</mu1>
+    <mu2>0.0</mu2>
     <kp>1000000.0</kp>
     <kd>100.0</kd>
     <minDepth>0.001</minDepth>
     <maxVel>1.0</maxVel>
-    <fdir1>1 0 0</fdir1>
     <material>Gazebo/FlatBlack</material>
-  </gazebo> -->
-     <gazebo reference="caster_bottom_back_link">
-        <mu1>0.0</mu1>
-        <mu2>0.0</mu2>
-        <kp>1000000.0</kp>
-        <kd>100.0</kd>
-        <minDepth>0.001</minDepth>
-        <maxVel>1.0</maxVel>
-        <material>Gazebo/FlatBlack</material>
-    </gazebo>
-  <!-- <gazebo reference="caster_top_back_link">
-    <mu1>0.1</mu1>
-    <mu2>0.1</mu2>
-    <kp>1000000.0</kp>
-    <kd>100.0</kd>
-    <minDepth>0.001</minDepth>
-    <maxVel>1.0</maxVel>
-    <fdir1>1 0 0</fdir1>
-    <material>Gazebo/FlatBlack</material>
-  </gazebo> -->
-   <gazebo reference="caster_top_back_link">
-        <mu1>0.0</mu1>
-        <mu2>0.0</mu2>
-        <kp>1000000.0</kp>
-        <kd>100.0</kd>
-        <minDepth>0.001</minDepth>
-        <maxVel>1.0</maxVel>
-        <material>Gazebo/FlatBlack</material>
-    </gazebo>
-  <!-- <gazebo>
-    <plugin name="differential_drive_controller" filename="libgazebo_ros_diff_drive.so">
-      <commandTopic>cmd_vel</commandTopic>
-      <odometryTopic>odom</odometryTopic>
-      <odometryFrame>odom</odometryFrame>
-      <odometrySource>world</odometrySource>
-      <publishOdomTF>true</publishOdomTF>
-      <robotBaseFrame>base_footprint</robotBaseFrame>
-      <publishWheelTF>false</publishWheelTF>
-      <publishTf>true</publishTf>
-      <publishWheelJointState>true</publishWheelJointState>
-      <legacyMode>false</legacyMode>
-      <updateRate>30</updateRate>
-      <leftJoint>wheel_left_joint</leftJoint>
-      <rightJoint>wheel_right_joint</rightJoint>
-      <topJoint>caster_top_back_joint</topJoint>
-      <bottomJoint>caster_bottom_back_joint</bottomJoint>
-      <wheelSeparation>0.160</wheelSeparation>
-      <wheelDiameter>0.066</wheelDiameter>
-      <wheelAcceleration>1</wheelAcceleration>
-      <wheelTorque>10</wheelTorque>
-      <rosDebugLevel>na</rosDebugLevel>
-    </plugin>
-  </gazebo> -->
+  </gazebo>
+  <gazebo reference="caster_top_back_link">
+      <mu1>0.0</mu1>
+      <mu2>0.0</mu2>
+      <kp>1000000.0</kp>
+      <kd>100.0</kd>
+      <minDepth>0.001</minDepth>
+      <maxVel>1.0</maxVel>
+      <material>Gazebo/FlatBlack</material>
+  </gazebo>
   <gazebo>
     <plugin name="differential_drive_controller" filename="libgazebo_ros_diff_drive.so">
@@ -99,5 +55,4 @@
       <odometryTopic>diff/odom</odometryTopic>
       <odometryFrame>odom</odometryFrame>
-      <!-- <robotBaseFrame>base_link</robotBaseFrame> -->
       <publishWheelTF>false</publishWheelTF>
       <publishOdomTF>true</publishOdomTF>

File: diff_drive/urdf/ddrive.urdf.xacro (robot description, xacro)
@@ -4,7 +4,9 @@
   <xacro:property name="ddrive" value="$(find diff_drive)/config/ddrive.yaml"/>
   <xacro:property name="dictionary" value="${load_yaml(ddrive)}"/>
-  <xacro:property name="L" value="${dictionary['L']}"/>
-  <xacro:property name="W" value="${dictionary['W']}"/>
-  <xacro:property name="H" value="${dictionary['H']}"/>
+  <xacro:property name="box_L" value="${dictionary['box_L']}"/>
+  <xacro:property name="box_W" value="${dictionary['box_W']}"/>
+  <xacro:property name="box_H" value="${dictionary['box_H']}"/>
+  <xacro:property name="box_mass" value="${dictionary['box_mass']}"/>
+    <xacro:property name="wheel_scale" value="${dictionary['wheel_scale']}"/>
   <material name="Black">
     <color rgba="0.0 0.0 0.0 1.0"/>
@@ -17,5 +19,5 @@
     <parent link="base_footprint"/>
     <child link="base_link"/>
-    <origin xyz="0 0 0.01" rpy="0 0 0"/>
+    <origin xyz="0 0 0" rpy="0 0 0"/>
   </joint>
   <link name="base_link">
@@ -23,5 +25,5 @@
       <origin xyz="0 0 0" rpy="0 0 0"/>
       <geometry>
-        <box size="${L} ${W} ${H}"/>
+        <box size="${box_L} ${box_W} ${box_H}"/>
       </geometry>
       <material name="light_black"/>
@@ -30,13 +32,13 @@
       <origin xyz="0 0 0" rpy="0 0 0"/>
       <geometry>
-        <box size="${L} ${W} ${H}"/>
+        <box size="${box_L} ${box_W} ${box_H}"/>
       </geometry>
     </collision>
     <inertial>
       <origin xyz="0 0 0" rpy="0 0 0"/>
-      <mass value="8.2573504e-01"/>
-      <inertia ixx="2.2124416e-03" ixy="-1.2294101e-05" ixz="3.4938785e-05"
-               iyy="2.1193702e-03" iyz="-5.0120904e-06"
-               izz="2.0064271e-03" />
+      <mass value="${box_mass}"/>
+      <inertia ixx="${box_mass*(box_W**2+box_H**2)/12}" ixy="0" ixz="0"
+               iyy="${box_mass*(box_L**2+box_H**2)/12}" iyz="0"
+               izz="${box_mass*(box_L**2+box_W**2)/12}"/>
     </inertial>
   </link>
@@ -44,5 +46,5 @@
     <parent link="base_link"/>
     <child link="wheel_left_link"/>
-    <origin xyz="${3*L/8} ${W/2 + 0.080} 0.0" rpy="-1.57 0 0"/>
+    <origin xyz="${3*box_L/8} ${box_W/2 + 0.080} 0.0" rpy="-1.57 0 0"/>
     <axis xyz="0 0 1"/>
   </joint>
@@ -51,5 +53,5 @@
       <origin xyz="0 0 0" rpy="1.57 0 0"/>
       <geometry>
-        <mesh filename="package://diff_drive/meshes/wheels/left_tire.stl" scale="0.005 0.005 0.005"/>
+        <mesh filename="package://diff_drive/meshes/wheels/left_tire.stl" scale="${wheel_scale*0.001} ${wheel_scale*0.001} ${wheel_scale*0.001}"/>
       </geometry>
       <material name="Black"/>
@@ -58,13 +60,13 @@
       <origin xyz="0 0 0" rpy="0 0 0"/>
       <geometry>
-        <cylinder length="0.09" radius="0.165"/>
+        <cylinder length="${wheel_scale*0.018}" radius="${wheel_scale*0.033}"/>
       </geometry>
     </collision>
     <inertial>
-      <origin xyz="0 0 0" />
-      <mass value="2.8498940e-02" />
-      <inertia ixx="1.1175580e-05" ixy="-4.2369783e-11" ixz="-5.9381719e-09"
-               iyy="1.1192413e-05" iyz="-1.4400107e-11"
-               izz="2.0712558e-05" />
+      <origin xyz="0 0 0" rpy="0 0 0"/>
+      <mass value="${wheel_scale*2.8498940e-02}" />
+      <inertia ixx="${(wheel_scale**3)*1.1175580e-05}" ixy="${(wheel_scale**3)*-4.2369783e-11}" ixz="${(wheel_scale**3)*-5.9381719e-09}"
+               iyy="${(wheel_scale**3)*1.1192413e-05}" iyz="${(wheel_scale**3)*-1.4400107e-11}"
+               izz="${(wheel_scale**3)*2.0712558e-05}" />
       </inertial>
   </link>
@@ -72,5 +74,5 @@
     <parent link="base_link"/>
     <child link="wheel_right_link"/>
-    <origin xyz="${3*L/8} ${-W/2 - 0.080} 0.0" rpy="-1.57 0 0"/>
+    <origin xyz="${3*box_L/8} ${-box_W/2 - 0.080} 0.0" rpy="-1.57 0 0"/>
     <axis xyz="0 0 1"/>
   </joint>
@@ -79,5 +81,5 @@
       <origin xyz="0 0 0" rpy="1.57 0 0"/>
       <geometry>
-        <mesh filename="package://diff_drive/meshes/wheels/right_tire.stl" scale="0.005 0.005 0.005"/>
+        <mesh filename="package://diff_drive/meshes/wheels/right_tire.stl" scale="${wheel_scale*0.001} ${wheel_scale*0.001} ${wheel_scale*0.001}"/>
       </geometry>
       <material name="Black"/>
@@ -86,13 +88,13 @@
       <origin xyz="0 0 0" rpy="0 0 0"/>
       <geometry>
-        <cylinder length="0.09" radius="0.165"/>
+        <cylinder length="${wheel_scale*0.018}" radius="${wheel_scale*0.033}"/>
       </geometry>
     </collision>
     <inertial>
-      <origin xyz="0 0 0" />
-      <mass value="2.8498940e-02" />
-      <inertia ixx="1.1175580e-05" ixy="-4.2369783e-11" ixz="-5.9381719e-09"
-               iyy="1.1192413e-05" iyz="-1.4400107e-11"
-               izz="2.0712558e-05" />
+      <origin xyz="0 0 0" rpy="0 0 0"/>
+      <mass value="${wheel_scale*2.8498940e-02}" />
+      <inertia ixx="${(wheel_scale**3)*1.1175580e-05}" ixy="${(wheel_scale**3)*-4.2369783e-11}" ixz="${(wheel_scale**3)*-5.9381719e-09}"
+               iyy="${(wheel_scale**3)*1.1192413e-05}" iyz="${(wheel_scale**3)*-1.4400107e-11}"
+               izz="${(wheel_scale**3)*2.0712558e-05}" />
       </inertial>
   </link>
@@ -100,5 +102,5 @@
     <parent link="base_link"/>
     <child link="caster_bottom_back_link"/>
-    <origin xyz="${-3*L/7} 0 ${-H/2 - 0.026}" rpy="-1.57 0 0"/>
+    <origin xyz="${-3*box_L/7} 0 ${-box_H/2 - 0.026}" rpy="-1.57 0 0"/>
   </joint>
   <link name="caster_bottom_back_link">
@@ -127,5 +129,5 @@
     <parent link="base_link"/>
     <child link="caster_top_back_link"/>
-    <origin xyz="${-3*L/7} 0 ${H/2 + 0.026}" rpy="-1.57 0 0"/>
+    <origin xyz="${-3*box_L/7} 0 ${box_H/2 + 0.026}" rpy="-1.57 0 0"/>
   </joint>
   <link name="caster_top_back_link">

Commit message: robot follows trajectory

File: diff_drive/urdf/ddrive.gazebo.xacro (robot description, xacro)
@@ -5,6 +5,6 @@
   </gazebo>
   <gazebo reference="wheel_left_link">
-    <mu1>0.3</mu1>
-    <mu2>0.3</mu2>
+    <mu1>0.5</mu1>
+    <mu2>0.5</mu2>
     <kp>500000.0</kp>
     <kd>10.0</kd>
@@ -15,6 +15,6 @@
   </gazebo>
   <gazebo reference="wheel_right_link">
-    <mu1>0.3</mu1>
-    <mu2>0.3</mu2>
+    <mu1>0.5</mu1>
+    <mu2>0.5</mu2>
     <kp>500000.0</kp>
     <kd>10.0</kd>
@@ -34,11 +34,11 @@
   </gazebo>
   <gazebo reference="caster_top_back_link">
-      <mu1>0.0</mu1>
-      <mu2>0.0</mu2>
-      <kp>1000000.0</kp>
-      <kd>100.0</kd>
-      <minDepth>0.001</minDepth>
-      <maxVel>1.0</maxVel>
-      <material>Gazebo/FlatBlack</material>
+    <mu1>0.0</mu1>
+    <mu2>0.0</mu2>
+    <kp>1000000.0</kp>
+    <kd>100.0</kd>
+    <minDepth>0.001</minDepth>
+    <maxVel>1.0</maxVel>
+    <material>Gazebo/FlatBlack</material>
   </gazebo>
   <gazebo>

File: diff_drive/urdf/ddrive.urdf.xacro (robot description, xacro)
@@ -46,5 +46,5 @@
     <parent link="base_link"/>
     <child link="wheel_left_link"/>
-    <origin xyz="${3*box_L/8} ${box_W/2 + 0.080} 0.0" rpy="-1.57 0 0"/>
+    <origin xyz="${-3*box_L/8} ${box_W/2 + 0.080} 0.0" rpy="-1.57 0 0"/>
     <axis xyz="0 0 1"/>
   </joint>
@@ -74,5 +74,5 @@
     <parent link="base_link"/>
     <child link="wheel_right_link"/>
-    <origin xyz="${3*box_L/8} ${-box_W/2 - 0.080} 0.0" rpy="-1.57 0 0"/>
+    <origin xyz="${-3*box_L/8} ${-box_W/2 - 0.080} 0.0" rpy="-1.57 0 0"/>
     <axis xyz="0 0 1"/>
   </joint>
@@ -102,5 +102,5 @@
     <parent link="base_link"/>
     <child link="caster_bottom_back_link"/>
-    <origin xyz="${-3*box_L/7} 0 ${-box_H/2 - 0.026}" rpy="-1.57 0 0"/>
+    <origin xyz="${3*box_L/7} 0 ${-box_H/2 - 0.026}" rpy="-1.57 0 0"/>
   </joint>
   <link name="caster_bottom_back_link">
@@ -129,5 +129,5 @@
     <parent link="base_link"/>
     <child link="caster_top_back_link"/>
-    <origin xyz="${-3*box_L/7} 0 ${box_H/2 + 0.026}" rpy="-1.57 0 0"/>
+    <origin xyz="${3*box_L/7} 0 ${box_H/2 + 0.026}" rpy="-1.57 0 0"/>
   </joint>
   <link name="caster_top_back_link">
