Commit message: add robot model

File: diff_drive/urdf/ddrive.urdf.xacro (robot description, xacro)
@@ -39,5 +39,5 @@
     <parent link="base_link"/>
     <child link="wheel_left_link"/>
-    <origin xyz="${L/4} ${W/2+0.080} 0.0" rpy="-1.57 0 0"/>
+    <origin xyz="${3*L/8} ${W/2 + 0.080} 0.0" rpy="-1.57 0 0"/>
     <axis xyz="0 0 1"/>
   </joint>
@@ -53,5 +53,5 @@
       <origin xyz="0 0 0" rpy="0 0 0"/>
       <geometry>
-        <cylinder length="0.018" radius="0.033"/>
+        <cylinder length="0.09" radius="0.165"/>
       </geometry>
     </collision>
@@ -67,5 +67,5 @@
     <parent link="base_link"/>
     <child link="wheel_right_link"/>
-    <origin xyz="${L/4} ${-W/2-0.080} 0.0" rpy="-1.57 0 0"/>
+    <origin xyz="${3*L/8} ${-W/2 - 0.080} 0.0" rpy="-1.57 0 0"/>
     <axis xyz="0 0 1"/>
   </joint>
@@ -81,5 +81,5 @@
       <origin xyz="0 0 0" rpy="0 0 0"/>
       <geometry>
-        <cylinder length="0.018" radius="0.033"/>
+        <cylinder length="0.09" radius="0.165"/>
       </geometry>
     </collision>
@@ -95,11 +95,18 @@
     <parent link="base_link"/>
     <child link="caster_bottom_back_link"/>
-    <origin xyz="${-L/4} 0 ${-H/2-0.020}" rpy="-1.57 0 0"/>
+    <origin xyz="${-3*L/7} 0 ${-H/2 - 0.030}" rpy="-1.57 0 0"/>
   </joint>
   <link name="caster_bottom_back_link">
+    <visual>
+      <origin rpy="1.57 0 0" xyz="0 0.001 0"/>
+      <geometry>
+        <sphere radius="0.03"/>
+      </geometry>
+      <material name="Black"/>
+    </visual>
     <collision>
-      <origin xyz="0 0.001 0" rpy="1.57 0 0"/>
+      <origin rpy="1.57 0 0" xyz="0 0.001 0"/>
       <geometry>
-        <box size="0.150 0.045 0.100"/>
+        <sphere radius="0.03"/>
       </geometry>
     </collision>
@@ -115,11 +122,18 @@
     <parent link="base_link"/>
     <child link="caster_top_back_link"/>
-    <origin xyz="${-L/4} 0 ${+H/2+0.020}" rpy="-1.57 0 0"/>
+    <origin xyz="${-3*L/7} 0 ${H/2 + 0.030}" rpy="-1.57 0 0"/>
   </joint>
   <link name="caster_top_back_link">
+    <visual>
+      <origin rpy="1.57 0 0" xyz="0 0.001 0"/>
+      <geometry>
+        <sphere radius="0.03"/>
+      </geometry>
+      <material name="Black"/>
+    </visual>
     <collision>
-      <origin xyz="0 0.001 0" rpy="1.57 0 0"/>
+      <origin rpy="1.57 0 0" xyz="0 0.001 0"/>
       <geometry>
-        <box size="0.150 0.045 0.100"/>
+        <sphere radius="0.03"/>
       </geometry>
     </collision>

Commit message: fixing color issues

File: diff_drive/urdf/ddrive.urdf.xacro (robot description, xacro)
@@ -7,4 +7,10 @@
   <xacro:property name="W" value="${dictionary['W']}"/>
   <xacro:property name="H" value="${dictionary['H']}"/>
+  <material name="Black">
+    <color rgba="0.0 0.0 0.0 1.0"/>
+  </material>
+  <material name="light_black">
+    <color rgba="0.2 0.2 0.2 1.0"/>
+  </material>
   <link name="base_footprint"/>
   <joint name="base_joint" type="fixed">
@@ -47,5 +53,5 @@
         <mesh filename="package://diff_drive/meshes/wheels/left_tire.stl" scale="0.005 0.005 0.005"/>
       </geometry>
-      <material name="dark"/>
+      <material name="Black"/>
     </visual>
     <collision>
@@ -75,5 +81,5 @@
         <mesh filename="package://diff_drive/meshes/wheels/right_tire.stl" scale="0.005 0.005 0.005"/>
       </geometry>
-      <material name="dark"/>
+      <material name="Black"/>
     </visual>
     <collision>

Commit message: flip_over node created. not working yet

File: diff_drive/urdf/ddrive.urdf.xacro (robot description, xacro)
@@ -8,5 +8,7 @@
   <xacro:property name="box_H" value="${dictionary['box_H']}"/>
   <xacro:property name="box_mass" value="${dictionary['box_mass']}"/>
-    <xacro:property name="wheel_scale" value="${dictionary['wheel_scale']}"/>
+  <xacro:property name="wheel_scale" value="${dictionary['wheel_scale']}"/>
+  <xacro:property name="caster_radius" value="${dictionary['caster_radius']}"/>
+  <xacro:property name="caster_mass" value="${dictionary['caster_mass']}"/>
   <material name="Black">
     <color rgba="0.0 0.0 0.0 1.0"/>
@@ -38,6 +40,6 @@
       <origin xyz="0 0 0" rpy="0 0 0"/>
       <mass value="${box_mass}"/>
-      <inertia ixx="${box_mass*(box_W**2+box_H**2)/12}" ixy="0" ixz="0"
-               iyy="${box_mass*(box_L**2+box_H**2)/12}" iyz="0"
+      <inertia ixx="${box_mass*(box_W**2+box_H**2)/12}" ixy="0.0" ixz="0.0"
+               iyy="${box_mass*(box_L**2+box_H**2)/12}" iyz="0.0"
                izz="${box_mass*(box_L**2+box_W**2)/12}"/>
     </inertial>
@@ -115,13 +117,13 @@
       <origin rpy="1.57 0 0" xyz="0 0 0"/>
       <geometry>
-        <sphere radius="0.03"/>
+        <sphere radius="${caster_radius}"/>
       </geometry>
     </collision>
     <inertial>
       <origin xyz="0 0 0" />
-      <mass value="0.005" />
-      <inertia ixx="0.001" ixy="0.0" ixz="0.0"
-               iyy="0.001" iyz="0.0"
-               izz="0.001" />
+      <mass value="${caster_mass}" />
+      <inertia ixx="${(2/5)*caster_mass*caster_radius**2}" ixy="0.0" ixz="0.0"
+               iyy="${(2/5)*caster_mass*caster_radius**2}" iyz="0.0"
+               izz="${(2/5)*caster_mass*caster_radius**2}" />
     </inertial>
   </link>
@@ -135,5 +137,5 @@
       <origin rpy="1.57 0 0" xyz="0 0 0"/>
       <geometry>
-        <sphere radius="0.03"/>
+        <sphere radius="${caster_radius}"/>
       </geometry>
       <material name="Black"/>
@@ -147,8 +149,8 @@
     <inertial>
       <origin xyz="0 0 0" />
-      <mass value="0.005" />
-      <inertia ixx="0.001" ixy="0.0" ixz="0.0"
-               iyy="0.001" iyz="0.0"
-               izz="0.001" />
+      <mass value="${caster_mass}" />
+      <inertia ixx="${(2/5)*caster_mass*caster_radius**2}" ixy="0.0" ixz="0.0"
+               iyy="${(2/5)*caster_mass*caster_radius**2}" iyz="0.0"
+               izz="${(2/5)*caster_mass*caster_radius**2}" />
     </inertial>
   </link>
